Commit message: phase 1 - gz teleop

File: src/donkey_description/urdf/donkey_car.urdf.xacro (robot description, xacro)
@@ -1,212 +1,9 @@
 <?xml version="1.0"?>
 <robot xmlns:xacro="http://www.ros.org/wiki/xacro" name="donkey_car">
-  <!-- ========================= -->
-  <!-- Parameters -->
-  <!-- ========================= -->
-  <xacro:property name="chassis_length" value="0.32"/>
-  <xacro:property name="chassis_width"  value="0.18"/>
-  <xacro:property name="chassis_height" value="0.06"/>
-  <xacro:property name="wheel_radius" value="0.033"/>
-  <xacro:property name="wheel_width"  value="0.025"/>
-  <xacro:property name="front_x" value="0.12"/>
-  <xacro:property name="rear_x"  value="-0.12"/>
-  <xacro:property name="left_y"  value="0.09"/>
-  <xacro:property name="right_y" value="-0.09"/>
-  <xacro:property name="base_z" value="${wheel_radius + chassis_height / 2.0}"/>
-  <!-- ========================= -->
-  <!-- Materials -->
-  <!-- ========================= -->
-  <material name="black">
-    <color rgba="0.02 0.02 0.02 1.0"/>
-  </material>
-  <material name="gray">
-    <color rgba="0.4 0.4 0.4 1.0"/>
-  </material>
-  <material name="blue">
-    <color rgba="0.1 0.3 0.9 1.0"/>
-  </material>
-  <material name="red">
-    <color rgba="0.9 0.1 0.1 1.0"/>
-  </material>
-  <!-- ========================= -->
-  <!-- Base Frames -->
-  <!-- ========================= -->
-  <!-- Ground projection frame -->
-  <link name="base_footprint"/>
-  <joint name="base_footprint_to_base_link" type="fixed">
-    <parent link="base_footprint"/>
-    <child link="base_link"/>
-    <origin xyz="0 0 ${base_z}" rpy="0 0 0"/>
-  </joint>
-  <!-- Main robot body frame -->
-  <link name="base_link">
-    <visual>
-      <origin xyz="0 0 0" rpy="0 0 0"/>
-      <geometry>
-        <box size="${chassis_length} ${chassis_width} ${chassis_height}"/>
-      </geometry>
-      <material name="blue"/>
-    </visual>
-    <collision>
-      <origin xyz="0 0 0" rpy="0 0 0"/>
-      <geometry>
-        <box size="${chassis_length} ${chassis_width} ${chassis_height}"/>
-      </geometry>
-    </collision>
-    <inertial>
-      <mass value="1.5"/>
-      <origin xyz="0 0 0"/>
-      <inertia
-        ixx="0.01" ixy="0.0" ixz="0.0"
-        iyy="0.02" iyz="0.0"
-        izz="0.02"/>
-    </inertial>
-  </link>
-  <!-- ========================= -->
-  <!-- Wheel Macro -->
-  <!-- ========================= -->
-  <xacro:macro name="wheel" params="name parent x y steerable">
-    <xacro:if value="${steerable}">
-      <!-- Steering pivot -->
-      <link name="${name}_steer_link">
-        <visual>
-          <geometry>
-            <box size="0.02 0.02 0.02"/>
-          </geometry>
-          <material name="gray"/>
-        </visual>
-        <collision>
-          <geometry>
-            <box size="0.02 0.02 0.02"/>
-          </geometry>
-        </collision>
-        <inertial>
-          <mass value="0.02"/>
-          <origin xyz="0 0 0"/>
-          <inertia
-            ixx="0.00000133" ixy="0.0" ixz="0.0"
-            iyy="0.00000133" iyz="0.0"
-            izz="0.00000133"/>
-        </inertial>
-      </link>
-      <joint name="${name}_steer_joint" type="revolute">
-        <parent link="${parent}"/>
-        <child link="${name}_steer_link"/>
-        <origin xyz="${x} ${y} ${-chassis_height / 2.0}" rpy="0 0 0"/>
-        <axis xyz="0 0 1"/>
-        <limit lower="-0.6" upper="0.6" effort="5.0" velocity="5.0"/>
-      </joint>
-      <link name="${name}_wheel_link">
-        <visual>
-          <!-- Cylinder axis is z by default; rotate so axle is along y -->
-          <origin xyz="0 0 0" rpy="1.5708 0 0"/>
-          <geometry>
-            <cylinder radius="${wheel_radius}" length="${wheel_width}"/>
-          </geometry>
-          <material name="black"/>
-        </visual>
-        <collision>
-          <origin xyz="0 0 0" rpy="1.5708 0 0"/>
-          <geometry>
-            <cylinder radius="${wheel_radius}" length="${wheel_width}"/>
-          </geometry>
-        </collision>
-        <inertial>
-          <mass value="0.05"/>
-          <origin xyz="0 0 0"/>
-          <inertia
-            ixx="0.00005" ixy="0.0" ixz="0.0"
-            iyy="0.00005" iyz="0.0"
-            izz="0.00005"/>
-        </inertial>
-      </link>
-      <joint name="${name}_wheel_joint" type="continuous">
-        <parent link="${name}_steer_link"/>
-        <child link="${name}_wheel_link"/>
-        <origin xyz="0 0 0" rpy="0 0 0"/>
-        <axis xyz="0 1 0"/>
-      </joint>
-    </xacro:if>
-    <xacro:unless value="${steerable}">
-      <link name="${name}_wheel_link">
-        <visual>
-          <origin xyz="0 0 0" rpy="1.5708 0 0"/>
-          <geometry>
-            <cylinder radius="${wheel_radius}" length="${wheel_width}"/>
-          </geometry>
-          <material name="black"/>
-        </visual>
-        <collision>
-          <origin xyz="0 0 0" rpy="1.5708 0 0"/>
-          <geometry>
-            <cylinder radius="${wheel_radius}" length="${wheel_width}"/>
-          </geometry>
-        </collision>
-        <inertial>
-          <mass value="0.05"/>
-          <origin xyz="0 0 0"/>
-          <inertia
-            ixx="0.00005" ixy="0.0" ixz="0.0"
-            iyy="0.00005" iyz="0.0"
-            izz="0.00005"/>
-        </inertial>
-      </link>
-      <joint name="${name}_wheel_joint" type="continuous">
-        <parent link="${parent}"/>
-        <child link="${name}_wheel_link"/>
-        <origin xyz="${x} ${y} ${-chassis_height / 2.0}" rpy="0 0 0"/>
-        <axis xyz="0 1 0"/>
-      </joint>
-    </xacro:unless>
-  </xacro:macro>
-  <!-- ========================= -->
-  <!-- Wheels -->
-  <!-- ========================= -->
-  <xacro:wheel name="front_left"  parent="base_link" x="${front_x}" y="${left_y}"  steerable="true"/>
-  <xacro:wheel name="front_right" parent="base_link" x="${front_x}" y="${right_y}" steerable="true"/>
-  <xacro:wheel name="rear_left"   parent="base_link" x="${rear_x}"  y="${left_y}"  steerable="false"/>
-  <xacro:wheel name="rear_right"  parent="base_link" x="${rear_x}"  y="${right_y}" steerable="false"/>
-  <!-- ========================= -->
-  <!-- Camera -->
-  <!-- ========================= -->
-  <link name="camera_link">
-    <visual>
-      <origin xyz="0 0 0" rpy="0 0 0"/>
-      <geometry>
-        <box size="0.035 0.025 0.025"/>
-      </geometry>
-      <material name="gray"/>
-    </visual>
-  </link>
-  <joint name="base_link_to_camera" type="fixed">
-    <parent link="base_link"/>
-    <child link="camera_link"/>
-    <origin xyz="0.14 0 0.07" rpy="0 0 0"/>
-  </joint>
-  <!-- ROS camera optical frame convention:
-       z forward, x right, y down
-  -->
-  <link name="camera_optical_frame"/>
-  <joint name="camera_link_to_camera_optical_frame" type="fixed">
-    <parent link="camera_link"/>
-    <child link="camera_optical_frame"/>
-    <origin xyz="0 0 0" rpy="-1.5708 0 -1.5708"/>
-  </joint>
-  <!-- ========================= -->
-  <!-- IMU -->
-  <!-- ========================= -->
-  <link name="imu_link">
-    <visual>
-      <origin xyz="0 0 0" rpy="0 0 0"/>
-      <geometry>
-        <box size="0.025 0.025 0.008"/>
-      </geometry>
-      <material name="gray"/>
-    </visual>
-  </link>
-  <joint name="base_link_to_imu" type="fixed">
-    <parent link="base_link"/>
-    <child link="imu_link"/>
-    <origin xyz="0 0 0.04" rpy="0 0 0"/>
-  </joint>
+  <xacro:include filename="$(find donkey_description)/urdf/donkey_base.xacro" />
+  <xacro:include filename="$(find donkey_description)/urdf/sensors/camera.xacro" />
+  <xacro:include filename="$(find donkey_description)/urdf/sensors/imu.xacro" />
+  <xacro:include filename="$(find donkey_sim)/urdf/ros2_control.xacro"/>
+  <xacro:donkey_camera parent="base_link" xyz="0.14 0 0.07" rpy="0 0 0" />
+  <xacro:donkey_imu    parent="base_link" xyz="0.0 0 0.04"  rpy="0 0 0" />
 </robot>
